Commit message: full code

File: src/scout_ros2/scout_description/urdf/scout_mini/scout_mini.urdf (robot description, URDF)
Before this commit: robot scout_mini, 8 links, 7 joints
Joints:
- joint os_lidar_mount: origin xyz=0.172248 -0.0012 0.1828 rpy=0 0 3.14 -> xyz=.178248 -0.0012 0.1828 rpy=0 0 3.14
